File: ibt2.kicad_pcb (KiCad board)
At the start: 2 copper layers, 48 x 62 mm, 24 parts, among them J1 SIGNAL, J2 BATTERY, J3 MOTOR, Q1 BTN8982TA, Q2 BTN8982TA, U1 SN74HC244DW

Commit message: ...
Parts:
- moved R6 25.5 mm to (131.9, 115.0)
- moved R3 17.9 mm to (143.2, 102.5), turned to 90 degrees
- moved D3 15.6 mm to (143.5, 116.3), turned to 90 degrees
- moved D2 14.6 mm to (149.9, 116.3), turned to 90 degrees
- moved R7 10.2 mm to (146.9, 103.0), turned to -90 degrees
- moved R1 8.17 mm to (143.2, 109.2), turned to -90 degrees
- moved R8 8.01 mm to (151.1, 110.6), turned to 90 degrees
- moved D1 6.23 mm to (138.4, 115.1), turned to 180 degrees
- moved J1 0.90 mm to (157.6, 103.3)
- moved G*** 0.44 mm to (120.7, 90.9)
Connections:
- J1 pad 2: LPWM -> RPWM
- J1 pad 3: RPWM -> LPWM
Routing:
- net +5V: track 84.7 -> 67.4 mm
- net Net-(D2-A): track 20.8 -> 4.39 mm
- net Net-(D1-A): track 4.14 -> 13.6 mm
- net LPWM: track 35.3 -> 27.2 mm
- net Net-(D3-A): track 18.0 -> 19.9 mm
- net RPWM: track 34.0 -> 32.7 mm
- net GND: vias 19 -> 18
Other:
- board size 48 x 62 mm -> 48 x 58.5 mm

Commit message: ....
Parts:
- moved R7 4.26 mm to (151.2, 102.9)
- moved R8 4.21 mm to (146.8, 110.5)
- moved R3 0.88 mm to (143.0, 103.3)
- moved R1 0.26 mm to (143.0, 109.1)
Routing:
- net Net-(D3-A): track 19.9 -> 12.0 mm
- net Net-(D2-A): track 4.39 -> 3.45 mm
